File: hardware/ago/ago.kicad_sch (KiCad schematic)
At the start: 3 parts

Commit message: finish hardware design.
Parts:
- added J?: Raspberry_Pi_2_3, symbol Connector:Raspberry_Pi_2_3
- added LS?: Speaker, symbol Device:Speaker
- added M_1, M_2, M_3, M_4, M_5, M_6: Motor_Servo, symbol Motor:Motor_Servo
- added U?: asr_pro, symbol Device:asr_pro
- added left_back, left_front, right_back, right_front: Motor_DC, symbol Motor:Motor_DC
- U?: value STM32F103C4Tx -> STM32F103C4Tx - MainController
Connections:
- net at U?.10 (LED4): now also M_5.1 (PWM)
- net at U?.11 (LED5): now also M_6.1 (PWM)
- net at U?.6 (LED0): now also M_1.1 (PWM)
- net at U?.7 (LED1): now also M_2.1 (PWM)
- net at U?.8 (LED2): now also M_3.1 (PWM)
- net at U?.9 (LED3): now also M_4.1 (PWM)
- net at U?.10 (IN3): now also U?.15 (PA5)
- net at U?.11 (EnB): now also U?.17 (PA7)
- net at U?.12 (IN4): now also U?.16 (PA6)
- net at U?.13 (OUT3): now also right_front.1 (+)
- net at U?.14 (OUT4): now also right_front.2 (-)
- net at U?.15 (OUT5): now also left_back.1 (+)
- net at U?.16 (OUT6): now also left_back.2 (-)
- net at U?.17 (OUT7): now also right_back.1 (+)
- net at U?.18 (OUT8): now also right_back.2 (-)
- net at U?.19 (IN5): now also U?.29 (PA8)
- net at U?.2 (OUT1): now also left_front.1 (+)
- net at U?.20 (IN6): now also U?.32 (PA11)
- net at U?.21 (EnC): now also U?.33 (PA12)
- net at U?.22 (IN7): now also U?.34 (PA13)
- net at U?.23 (IN8): now also U?.37 (PA14)
- net at U?.24 (EnD): now also U?.38 (PA15)
- net at U?.3 (OUT2): now also left_front.2 (-)
- net at U?.5 (ENA): now also U?.12 (PA2)
- net at U?.6 (IN2): now also U?.14 (PA4)
- net at U?.7 (IN1): now also U?.13 (PA3)
- net GND: now reaches U?.8 (GND)
- net VCC: now reaches U?.9 (Vss)
- new net: LS?.1, U?. (VCC_5V)
- new net: LS?.2, U?. (VCC_5V)

Commit message: fix hardware design.
Parts:
- added MK?: Microphone_Crystal, symbol Device:Microphone_Crystal
