File: hardware/pcb_design/ago.kicad_sch (KiCad schematic)
At the start: 21 parts

Commit message: refresh hardware design.
Parts:
- removed MK?: Microphone_Crystal, symbol Device:Microphone_Crystal
- removed U?: OpenMV, symbol Video:OpenMV
- removed U?: ESP8266EX, Package_DFN_QFN:QFN-32-1EP_5x5mm_P0.5mm_EP3.45x3.45mm, symbol MCU_Espressif:ESP8266EX
- removed U?: oled-9.6, symbol Display_Graphic:oled-9.6
- removed U?: MPU6050, symbol Display_Graphic:MPU6050
- removed U?: asr_pro, symbol Device:asr_pro
- removed U?: GY-530_VL53L0X, symbol Video:GY-530_VL53L0X
- added U1: ESP32-S3, Package_DFN_QFN:QFN-56-1EP_7x7mm_P0.4mm_EP4x4mm, symbol MCU_Espressif:ESP32-S3
- added U2: (no value), symbol New_Library:JQ6500
Connections:
- net at LS?.1: now also U2. (RX)
- net at LS?.2: now also U2. (RX)
- net at U?.11 (EnB): now also U?.18 (PB0), U?.5 (ENA)
- net at U?.21 (EnC): now also U?.19 (PB1), U?.24 (EnD)
- net at U?.6 (IN2): no longer U?.31 (PA10-RX1)
- net at U?.12 (PA2-TX2): now also U2. (RX)
- net at U?.13 (PA3-RX2): now also U2. (RX)
- new net: U1.2 (VDD3P3), U1.3 (VDD3P3)
- new net: U1.55 (VDDA), U1.56 (VDDA)
Other:
- moved on the sheet: M_1, M_2, M_3, M_4, M_5, M_6, U?, left_back, left_front, right_back, right_front

Commit message: fix hardware design to 43,44 GPIO.
Connections:
- net at U2. (RX): now also U?.13 (PA3-RX2)
Changed lines of the file:
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@@
+		)
+	)
+	(bus
+		(pts
+			(xy 50.8 107.95) (xy 57.15 107.95)
+		)
+		(stroke
+			(width 0)
+			(type default)
 		)
 	)
@@
 		)
 	)
+	(bus
+		(pts
+			(xy 53.34 105.41) (xy 57.15 105.41)
+		)
+		(stroke
+			(width 0)
+			(type default)
+		)
+	)
 	(wire
 		(pts
@@
 		)
 	)
+	(bus
+		(pts
+			(xy 50.8 36.83) (xy 50.8 107.95)
+		)
+		(stroke
+			(width 0)
+			(type default)
+		)
+	)
 	(wire
 		(pts
@@
 		)
 	)
+	(bus
+		(pts
+			(xy 111.76 95.25) (xy 111.76 133.35)
+		)
+		(stroke
+			(width 0)
+			(type default)
+		)
+	)
 	(wire
 		(pts
@@
 		)
 	)
-	(bus
-		(pts
-			(xy 102.87 97.79) (xy 106.68 97.79)
-		)
-		(stroke
-			(width 0)
-			(type default)
-		)
-	)
 	(wire
 		(pts
@@
 	(wire
 		(pts
-			(xy 125.73 95.25) (xy 127 95.25)
-		)
-		(stroke
-			(width 0)
-			(type default)
-		)
-	)
-	(wire
-		(pts
 			(xy 151.13 128.27) (xy 151.13 124.46)
 		)
@@
 		)
 	)
-	(bus
-		(pts
-			(xy 106.68 97.79) (xy 106.68 92.71)
-		)
-		(stroke
-			(width 0)
-			(type default)
-		)
-	)
 	(wire
 		(pts
@@
 		)
 	)
-	(bus
-		(pts
-			(xy 102.87 95.25) (xy 128.27 95.25)
-		)
-		(stroke
-			(width 0)
-			(type default)
-		)
-	)
 	(wire
 		(pts
@@
 		)
 	)
+	(bus
+		(pts
+			(xy 53.34 133.35) (xy 53.34 105.41)
+		)
+		(stroke
+			(width 0)
+			(type default)
+		)
+	)
 	(wire
 		(pts
@@
 		)
 	)
+	(bus
+		(pts
+			(xy 106.68 92.71) (xy 106.68 36.83)
+		)
+		(stroke
+			(width 0)
+			(type default)
+		)
+	)
 	(wire
 		(pts
@@
 		)
 	)
+	(bus
+		(pts
+			(xy 111.76 133.35) (xy 53.34 133.35)
+		)
+		(stroke
+			(width 0)
+			(type default)
+		)
+	)
 	(wire
 		(pts
@@
 		)
 	)
+	(bus
+		(pts
+			(xy 106.68 36.83) (xy 50.8 36.83)
+		)
+		(stroke
+			(width 0)
+			(type default)
+		)
+	)
 	(wire
 		(pts
@@
 		)
 		(stroke
+			(width 0)
+			(type default)
+		)
+	)
+	(bus
+		(pts
+			(xy 125.73 95.25) (xy 111.76 95.25)
+		)
+		(stroke
