File: hardware/pcb_design/ago.kicad_sch (KiCad schematic)
At the start: 16 parts, among them U1 ESP32-S3

Commit message: fix hardware design.
Connections:
- net at U2. (RX): now also U?.13 (PA3-RX2)
Changed lines of the file:
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@@
+		)
+	)
+	(bus
+		(pts
+			(xy 102.87 59.69) (xy 105.41 59.69)
+		)
+		(stroke
+			(width 0)
+			(type default)
 		)
 	)
@@
 		)
 	)
-	(bus
-		(pts
-			(xy 50.8 107.95) (xy 57.15 107.95)
-		)
-		(stroke
-			(width 0)
-			(type default)
-		)
-	)
 	(wire
 		(pts
@@
 	(bus
 		(pts
-			(xy 53.34 105.41) (xy 57.15 105.41)
+			(xy 105.41 46.99) (xy 105.41 59.69)
 		)
 		(stroke
@@
 	(bus
 		(pts
-			(xy 50.8 36.83) (xy 50.8 107.95)
+			(xy 102.87 100.33) (xy 109.22 100.33)
 		)
 		(stroke
@@
 		)
 	)
-	(bus
-		(pts
-			(xy 111.76 95.25) (xy 111.76 133.35)
-		)
-		(stroke
-			(width 0)
-			(type default)
-		)
-	)
 	(wire
 		(pts
@@
 		)
 	)
+	(bus
+		(pts
+			(xy 101.6 45.72) (xy 106.68 45.72)
+		)
+		(stroke
+			(width 0)
+			(type default)
+		)
+	)
 	(wire
 		(pts
@@
 		)
 	)
-	(bus
-		(pts
-			(xy 109.22 100.33) (xy 109.22 127)
-		)
-		(stroke
-			(width 0)
-			(type default)
-		)
-	)
 	(wire
 		(pts
@@
 		)
 	)
-	(bus
-		(pts
-			(xy 102.87 124.46) (xy 106.68 124.46)
-		)
-		(stroke
-			(width 0)
-			(type default)
-		)
-	)
 	(wire
 		(pts
@@
 		)
 	)
+	(bus
+		(pts
+			(xy 106.68 45.72) (xy 106.68 62.23)
+		)
+		(stroke
+			(width 0)
+			(type default)
+		)
+	)
 	(wire
 		(pts
@@
 		)
 	)
-	(bus
-		(pts
-			(xy 53.34 133.35) (xy 53.34 105.41)
-		)
-		(stroke
-			(width 0)
-			(type default)
-		)
-	)
 	(wire
 		(pts
@@
 	(bus
 		(pts
-			(xy 106.68 92.71) (xy 106.68 36.83)
+			(xy 101.6 46.99) (xy 105.41 46.99)
 		)
 		(stroke
@@
 		)
 	)
-	(bus
-		(pts
-			(xy 111.76 133.35) (xy 53.34 133.35)
-		)
-		(stroke
-			(width 0)
-			(type default)
-		)
-	)
 	(wire
 		(pts
@@
 		)
 	)
+	(bus
+		(pts
+			(xy 106.68 92.71) (xy 106.68 102.87)
+		)
+		(stroke
+			(width 0)
+			(type default)
+		)
+	)
 	(wire
 		(pts
@@
 		)
 	)
-	(bus
-		(pts
-			(xy 106.68 36.83) (xy 50.8 36.83)
-		)
-		(stroke
-			(width 0)
-			(type default)
-		)
-	)
 	(wire
 		(pts
@@
 	(bus
 		(pts
-			(xy 106.68 102.87) (xy 106.68 124.46)
+			(xy 109.22 95.25) (xy 109.22 100.33)
 		)
 		(stroke
@@
 		)
 	)
+	(bus
+		(pts
+			(xy 125.73 95.25) (xy 109.22 95.25)
+		)
+		(stroke
+			(width 0)
+			(type default)
+		)
+	)
 	(wire
 		(pts
@@
 		)
 	)
+	(bus
+		(pts
+			(xy 102.87 62.23) (xy 106.68 62.23)
+		)
+		(stroke
+			(width 0)
+			(type default)
+		)
+	)
 	(wire
 		(pts
@@
 		)
 	)
-	(bus
-		(pts
-			(xy 102.87 127) (xy 109.22 127)
-		)
-		(stroke
-			(width 0)
-			(type default)
-		)
-	)
 	(wire
 		(pts
@@
 		)
 	)
-	(bus
-		(pts
-			(xy 102.87 100.33) (xy 109.22 100.33)
-		)
-		(stroke
-			(width 0)
-			(type default)
-		)
-	)
 	(wire
 		(pts
@@
 		(pts
 			(xy 123.19 115.57) (xy 184.15 115.57)
-		)
-		(stroke
-			(width 0)
-			(type default)
-		)
-	)
-	(bus
-		(pts
-			(xy 125.73 95.25) (xy 111.76 95.25)
 		)
 		(stroke
@@
 	)
 	(image
-		(at 99.06 124.46)
+		(at 97.79 48.26)
 		(scale 3.52778)
 		(data "iVBORw0KGgoAAAANSUhEUgAAACYAAAAnCAYAAABjYToLAAAABHNCSVQICAgIfAhkiAAADelJREFU"
